File: Yolk Workshop - Germinal Disc/Controller.kicad_sch (KiCad schematic)
At the start: 9 parts, among them J1 FFC2B35-50-G_REVA2, J2 046809610110846, U1 LTR-303ALS-01

Commit message: updates to HIP and Controller design
Parts:
- removed C1: 100n, Capacitor_SMD:C_0402_1005Metric_Pad0.74x0.62mm_HandSolder, symbol Device:C
- removed R3: 3k6, Resistor_SMD:R_0402_1005Metric_Pad0.72x0.64mm_HandSolder, symbol Device:R_Small
- removed U1: LTR-303ALS-01, OptoDevice:Lite-On_LTR-303ALS-01, symbol Sensor_Optical:LTR-303ALS-01
- added C1: 100n, Capacitor_SMD:C_0603_1608Metric, symbol Device:C_Small
- added SW1: POWER_SW, Button_Switch_SMD:SW_SPDT_CK_JS102011SAQN, symbol Switch:SW_SPDT
- R1: value 0R -> RSET2; footprint Resistor_SMD:R_0402_1005Metric -> Resistor_SMD:R_0603_1608Metric_Pad0.98x0.95mm_HandSolder
- R2: value 0R -> RSET; footprint Resistor_SMD:R_0402_1005Metric -> Resistor_SMD:R_0603_1608Metric_Pad0.98x0.95mm_HandSolder
- R28, R29: footprint Resistor_SMD:R_0402_1005Metric -> Resistor_SMD:R_0402_1005Metric_Pad0.72x0.64mm_HandSolder
Connections:
- net AMB_I2C_SCL is gone; now on net +3.3V: R1.1
- net LMAT_INT is gone; now on net LMAT_SDB: J1.45
- net LMAT_RST is gone; now on net EXT_ALRT: J1.46
- net +3.3V: no longer J2.1 (Pin_1)
- net EXT_ALRT: no longer J1.49
- net GND: now also R2.2, C1.2; no longer J1.50
- net LMAT_SCL: no longer R1.2
- net LMAT_SDA: no longer R2.2
- net LMAT_SDB: no longer J1.47
- net AMB_I2C_INT renamed SW_A
- net SW_A: now also SW1.2 (B)
- net AMB_I2C_SDA renamed BRD_VERSION
- net BRD_VERSION: now also J1.49, R1.2, C1.1
- new net PS_BRD_VERSION: J1.50, J2.1 (Pin_1)
- new net SW_B: J1.47, SW1.1 (A)
- no-connect marks 0 -> 1
Other:
- note added: "Controller Connector"
- note added: "Power Switch"
- note added: "Proximity Sensor Connector"
