File: Yolk Workshop - Germinal Disc/Key Matrix.kicad_sch (KiCad schematic)
At the start: 246 parts, among them K1 ESC, K10 F9, K11 F10, K12 F11, K13 F12, K14 DEL/LOCK, K15 §[±], K16 1[!], K17 2[@], K18 3[£]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

Commit message: updates to HIP and Controller design
Parts:
- removed R4, R5, R6, R7, R8, R9: 25k, Resistor_SMD:R_0402_1005Metric_Pad0.72x0.64mm_HandSolder, symbol Device:R_Small
