File: Yolk Workshop - Germinal Disc/L_MAT.kicad_sch (KiCad schematic)
At the start: 110 parts, among them U2 IS31FL3737-QFLS4-TR

Commit message: updates to HIP and Controller design
Parts:
- removed C80: 100n, Capacitor_SMD:C_0402_1005Metric_Pad0.74x0.62mm_HandSolder, symbol Device:C
- removed D100, D101, D102, D103, D104, D105, D106, D107, D108, D109, D110, D111, D112, D113, D114, D115, D116, D117, D118, D119, D120, D121, D122, D123, D124, D125, D126, D127, D128, D129, D130, D131, D132, D133, D134, D135, D136, D137, D138, D139, D140, D141, D142, D143, D144, D145, D146, D147, D148, D149, D150, D151, D152, D153, D154, D155, D156, D157, D158, D159, D160, D161, D162, D79, D80, D81, D82, D83, D84, D85, D86, D87, D88, D89, D90, D91, D92, D93, D94, D95, D96, D97, D98, D99: KW EELP41.RU, LED_SMD:LED_0603_1608Metric, symbol Device:LED_Small_Filled
- removed R10, R11: 2k2, Resistor_SMD:R_0402_1005Metric_Pad0.72x0.64mm_HandSolder, symbol Device:R_Small
- removed R12, R23: 100k, Resistor_SMD:R_0402_1005Metric_Pad0.72x0.64mm_HandSolder, symbol Device:R
- removed R13, R15, R16, R17, R18, R19, R20, R21, R22, R25, R26, R27: 0R, Resistor_SMD:R_0402_1005Metric_Pad0.72x0.64mm_HandSolder, symbol Device:R
- removed U2: IS31FL3737-QFLS4-TR, picostroke:QFN40P500X500X80-41N-D, symbol IS31FL3737-QFLS4-TR:IS31FL3737-QFLS4-TR
- added C86: 470n, Capacitor_SMD:C_0402_1005Metric_Pad0.74x0.62mm_HandSolder, symbol Device:C
- added C89, C90: 100n, Capacitor_SMD:C_0402_1005Metric_Pad0.74x0.62mm_HandSolder, symbol Device:C
- added D100, D101, D102, D103, D104, D105, D106, D107, D108, D109, D110, D111, D112, D113, D114, D115, D116, D117, D118, D119, D120, D121, D122, D123, D124, D125, D126, D127, D128, D129, D130, D131, D132, D133, D134, D135, D136, D139, D140, D141, D142, D143, D144, D145, D146, D147, D148, D149, D154, D155, D156, D157, D158, D159, D160, D161, D162, D165, D166, D79, D80, D81, D82, D83, D84, D85, D86, D87, D88, D89, D90, D91, D92, D93, D94, D95, D96, D97, D98, D99: IN-S128TATRGB, picostroke:3228 RBG_LED, symbol Device:LED_ARBG
- added R10: 10K, Resistor_SMD:R_0603_1608Metric_Pad0.98x0.95mm_HandSolder, symbol Device:R
- added R12, R13, R15, R16, R18, R19, R21, R22, R24, R25, R27, R30, R32, R33, R35, R36, R38, R39, R44, R45: 51R, Resistor_SMD:R_0402_1005Metric_Pad0.72x0.64mm_HandSolder, symbol Device:R_Small
- added R14, R17, R20, R23, R26, R31, R34, R37, R40, R46: 20R, Resistor_SMD:R_0402_1005Metric_Pad0.72x0.64mm_HandSolder, symbol Device:R_Small
- added U1, U2: IS31FL3743A-QULS4-TR, picostroke:QFN40P500X500X60-41N-D, symbol IS31FL3743A:IS31FL3743A-QULS4-TR
- C80: renamed from C81; footprint Capacitor_SMD:C_0402_1005Metric_Pad0.74x0.62mm_HandSolder -> Capacitor_SMD:C_0603_1608Metric
- C85: value 100n -> 22u; footprint Capacitor_SMD:C_0402_1005Metric_Pad0.74x0.62mm_HandSolder -> Capacitor_SMD:C_0603_1608Metric_Pad1.08x0.95mm_HandSolder
- R11: renamed from R24; value 140k -> 10K; footprint Resistor_SMD:R_0402_1005Metric_Pad0.72x0.64mm_HandSolder -> Resistor_SMD:R_0603_1608Metric_Pad0.98x0.95mm_HandSolder
- renumbered C82 to C81, C83 to C82, C84 to C83, C86 to C92, R14 to R3
Connections:
- net +5V: now also C85.1, C86.1, C89.2, C90.2, U1.22 (VCC), U1.24 (ADDR2), U1.5 (PVCC), U2.22 (VCC), U2.5 (PVCC); no longer C85.2
- net GND: now also C85.2, C86.2, C89.1, C90.1, R10.1, U1.16 (PGND), U1.23 (GND), U1.25 (ADDR1), U1.41 (EP), U2.16 (PGND), U2.23 (GND), U2.24 (ADDR2), U2.25 (ADDR1), U2.41 (EP); no longer C85.1
- net LMAT_SCL: now also U1.27 (SCL), U2.27 (SCL)
- net LMAT_SDA: now also U1.28 (SDA), U2.28 (SDA)
- net LMAT_SDB: now also U1.26 (SDB), U2.26 (SDB)
- net LMAT_REXT renamed LMAT_REXT_x
- net LMAT_REXT_x: now also U2.29 (ISET)
- new net: D124.2 (RK), D125.2 (RK), D126.2 (RK), D127.2 (RK), D128.2 (RK), D129.2 (RK), D130.2 (RK), D131.2 (RK), D132.2 (RK), D133.2 (RK), D134.2 (RK), R34.1
- new net: D124.3 (BK), D125.3 (BK), D126.3 (BK), D127.3 (BK), D128.3 (BK), D129.3 (BK), D130.3 (BK), D131.3 (BK), D132.3 (BK), D133.3 (BK), D134.3 (BK), R32.1
- new net: D124.4 (GK), D125.4 (GK), D126.4 (GK), D127.4 (GK), D128.4 (GK), D129.4 (GK), D130.4 (GK), D131.4 (GK), D132.4 (GK), D133.4 (GK), D134.4 (GK), R33.1
- new net: D90.2 (RK), D91.2 (RK), D92.2 (RK), D93.2 (RK), R14.1
- new net: D120.2 (RK), D121.2 (RK), D122.2 (RK), D123.2 (RK), R31.1
- new net: D120.3 (BK), D121.3 (BK), D122.3 (BK), D123.3 (BK), R27.1
- new net: D120.4 (GK), D121.4 (GK), D122.4 (GK), D123.4 (GK), R30.1
- new net: D154.2 (RK), D155.2 (RK), D156.2 (RK), D157.2 (RK), D158.2 (RK), D159.2 (RK), D160.2 (RK), D161.2 (RK), D162.2 (RK), D165.2 (RK), D166.2 (RK), R46.1
- new net: D154.3 (BK), D155.3 (BK), D156.3 (BK), D157.3 (BK), D158.3 (BK), D159.3 (BK), D160.3 (BK), D161.3 (BK), D162.3 (BK), D165.3 (BK), D166.3 (BK), R44.1
- new net: D154.4 (GK), D155.4 (GK), D156.4 (GK), D157.4 (GK), D158.4 (GK), D159.4 (GK), D160.4 (GK), D161.4 (GK), D162.4 (GK), D165.4 (GK), D166.4 (GK), R45.1
- new net: D135.2 (RK), D136.2 (RK), R37.1
- new net: D105.3 (BK), D106.3 (BK), D107.3 (BK), D108.3 (BK), R21.1
- new net: D105.4 (GK), D106.4 (GK), D107.4 (GK), D108.4 (GK), R22.1
- new net: D79.2 (RK), D80.2 (RK), D81.2 (RK), D82.2 (RK), D83.2 (RK), D84.2 (RK), D85.2 (RK), D86.2 (RK), D87.2 (RK), D88.2 (RK), D89.2 (RK), R17.1
- new net: D79.3 (BK), D80.3 (BK), D81.3 (BK), D82.3 (BK), D83.3 (BK), D84.3 (BK), D85.3 (BK), D86.3 (BK), D87.3 (BK), D88.3 (BK), D89.3 (BK), R15.1
- new net: D79.4 (GK), D80.4 (GK), D81.4 (GK), D82.4 (GK), D83.4 (GK), D84.4 (GK), D85.4 (GK), D86.4 (GK), D87.4 (GK), D88.4 (GK), D89.4 (GK), R16.1
- new net: D100.2 (RK), D101.2 (RK), D102.2 (RK), D103.2 (RK), D104.2 (RK), D94.2 (RK), D95.2 (RK), D96.2 (RK), D97.2 (RK), D98.2 (RK), D99.2 (RK), R20.1
- new net: D100.3 (BK), D101.3 (BK), D102.3 (BK), D103.3 (BK), D104.3 (BK), D94.3 (BK), D95.3 (BK), D96.3 (BK), D97.3 (BK), D98.3 (BK), D99.3 (BK), R18.1
- new net: D100.4 (GK), D101.4 (GK), D102.4 (GK), D103.4 (GK), D104.4 (GK), D94.4 (GK), D95.4 (GK), D96.4 (GK), D97.4 (GK), D98.4 (GK), D99.4 (GK), R19.1
- new net: D109.2 (RK), D110.2 (RK), D111.2 (RK), D112.2 (RK), D113.2 (RK), D114.2 (RK), D115.2 (RK), D116.2 (RK), D117.2 (RK), D118.2 (RK), D119.2 (RK), R26.1
- new net: D135.3 (BK), D136.3 (BK), R35.1
- new net: D135.4 (GK), D136.4 (GK), R36.1
- new net: D109.4 (GK), D110.4 (GK), D111.4 (GK), D112.4 (GK), D113.4 (GK), D114.4 (GK), D115.4 (GK), D116.4 (GK), D117.4 (GK), D118.4 (GK), D119.4 (GK), R25.1
- new net: D90.3 (BK), D91.3 (BK), D92.3 (BK), D93.3 (BK), R12.1
- new net: D90.4 (GK), D91.4 (GK), D92.4 (GK), D93.4 (GK), R13.1
- new net: D139.4 (GK), D140.4 (GK), D141.4 (GK), D142.4 (GK), D143.4 (GK), D144.4 (GK), D145.4 (GK), D146.4 (GK), D147.4 (GK), D148.4 (GK), D149.4 (GK), R39.1
- new net: D139.2 (RK), D140.2 (RK), D141.2 (RK), D142.2 (RK), D143.2 (RK), D144.2 (RK), D145.2 (RK), D146.2 (RK), D147.2 (RK), D148.2 (RK), D149.2 (RK), R40.1
- new net: D139.3 (BK), D140.3 (BK), D141.3 (BK), D142.3 (BK), D143.3 (BK), D144.3 (BK), D145.3 (BK), D146.3 (BK), D147.3 (BK), D148.3 (BK), D149.3 (BK), R38.1
- new net: D105.2 (RK), D106.2 (RK), D107.2 (RK), D108.2 (RK), R23.1
- new net: D109.3 (BK), D110.3 (BK), D111.3 (BK), D112.3 (BK), D113.3 (BK), D114.3 (BK), D115.3 (BK), D116.3 (BK), D117.3 (BK), D118.3 (BK), D119.3 (BK), R24.1
- new net COL10x: R24.2, U2.21 (CS10)
- new net COL10y: R12.2, U1.21 (CS10)
- new net COL11x: R25.2, U2.20 (CS11)
- new net COL11y: R13.2, U1.20 (CS11)
- new net COL12x: R26.2, U2.19 (CS12)
- new net COL12y: R14.2, U1.19 (CS12)
- new net COL13x: R18.2, U2.18 (CS13)
- new net COL14x: R19.2, U2.17 (CS14)
- new net COL15x: R20.2, U2.15 (CS15)
- new net COL16x: R15.2, U2.14 (CS16)
- new net COL17x: R16.2, U2.13 (CS17)
- new net COL18x: R17.2, U2.12 (CS18)
- new net COL1x: R44.2, U2.39 (CS1)
- new net COL1y: R35.2, U1.39 (CS1)
- new net COL2x: R45.2, U2.38 (CS2)
- new net COL2y: R36.2, U1.38 (CS2)
- new net COL3x: R46.2, U2.37 (CS3)
- new net COL3y: R37.2, U1.37 (CS3)
- new net COL4x: R38.2, U2.36 (CS4)
- new net COL4y: R27.2, U1.36 (CS4)
- new net COL5x: R39.2, U2.35 (CS5)
- new net COL5y: R30.2, U1.35 (CS5)
- new net COL6x: R40.2, U2.34 (CS6)
- new net COL6y: R31.2, U1.34 (CS6)
- new net COL7x: R32.2, U2.33 (CS7)
- new net COL7y: R21.2, U1.33 (CS7)
- new net COL8x: R33.2, U2.32 (CS8)
- new net COL8y: R22.2, U1.32 (CS8)
- new net COL9x: R34.2, U2.31 (CS9)
- new net COL9y: R23.2, U1.31 (CS9)
- new net LMAT_REXT_y: R10.2, U1.29 (ISET)
- new net ROW10x: D110.1 (A), D125.1 (A), D140.1 (A), D155.1 (A), D80.1 (A), D95.1 (A), U2.40 (SW10)
- new net ROW11x: D109.1 (A), D124.1 (A), D139.1 (A), D154.1 (A), D79.1 (A), D94.1 (A), U2.11 (SW11)
- new net ROW1x: D104.1 (A), D119.1 (A), D134.1 (A), D149.1 (A), D166.1 (A), D89.1 (A), U2.6 (SW1)
- new net ROW1y: D108.1 (A), D123.1 (A), D93.1 (A), U1.6 (SW1)
- new net ROW2x: D103.1 (A), D118.1 (A), D133.1 (A), D148.1 (A), D165.1 (A), D88.1 (A), U2.4 (SW2)
- new net ROW2y: D107.1 (A), D122.1 (A), D92.1 (A), U1.4 (SW2)
- new net ROW3x: D102.1 (A), D117.1 (A), D132.1 (A), D147.1 (A), D162.1 (A), D87.1 (A), U2.7 (SW3)
- new net ROW3y: D106.1 (A), D121.1 (A), D136.1 (A), D91.1 (A), U1.7 (SW3)
- new net ROW4x: D101.1 (A), D116.1 (A), D131.1 (A), D146.1 (A), D161.1 (A), D86.1 (A), U2.3 (SW4)
- new net ROW4y: D105.1 (A), D120.1 (A), D135.1 (A), D90.1 (A), U1.3 (SW4)
- new net ROW5x: D100.1 (A), D115.1 (A), D130.1 (A), D145.1 (A), D160.1 (A), D85.1 (A), U2.8 (SW5)
- new net ROW6x: D114.1 (A), D129.1 (A), D144.1 (A), D159.1 (A), D84.1 (A), D99.1 (A), U2.2 (SW6)
- new net ROW7x: D113.1 (A), D128.1 (A), D143.1 (A), D158.1 (A), D83.1 (A), D98.1 (A), U2.9 (SW7)
- new net ROW8x: D112.1 (A), D127.1 (A), D142.1 (A), D157.1 (A), D82.1 (A), D97.1 (A), U2.1 (SW8)
- new net ROW9x: D111.1 (A), D126.1 (A), D141.1 (A), D156.1 (A), D81.1 (A), D96.1 (A), U2.10 (SW9)
- new net SYNC: U1.30 (SYNC), U2.30 (SYNC)
- no-connect marks 6 -> 13
Other:
- note removed: "ALT LED [YELLOW]: APDA3020LSYCK/J3-PF"
- note removed: "LED Resistor Calculation [ OPTIONAL ]"
- note removed: "Max LED Current & Power"
- moved on the sheet: C80, C81, C82, C83, C92, R11, R3
