File: Yolk Workshop - Vitellus/FPC.kicad_sch (KiCad schematic)
At the start: 1 part, among them J6 FFC2B35-50-G_REVA2

Commit message: updates to HIP and Controller design
Parts:
- added TP11, TP12, TP13, TP14, TP15: TestPoint, TestPoint:TestPoint_Pad_D1.0mm, symbol Connector:TestPoint
Connections:
- net LMAT_INT is gone; now on net LMAT_SDB: J6.45
- net LMAT_RST is gone; now on net PROX_I2C_INT: J6.46
- net GND: no longer J6.50
- net LMAT_SCL: now also TP13.1
- net LMAT_SDA: now also TP14.1
- net LMAT_SDB: now also TP15.1; no longer J6.47
- net PROX_I2C_INT: no longer J6.49
- net AMB_I2C_INT renamed PWR_SW_A
- new net KB_VER: J6.49, TP11.1
- new net PS_VER: J6.50, TP12.1
- new net PWR_SW_B: J6.47
Other:
- company: (none) -> Yolk Workshop
