File: Yolk Workshop - Vitellus/MCU.kicad_sch (KiCad schematic)
At the start: 54 parts, among them J2 Conn_ARM_JTAG_SWD_10, J4 BLE_DBG, J5 UART, J7 51281-1298, SW1 ~{BOOT}, SW2 ~{RESET}, SW3 BT_SCAN, U2 M24512E-FMN6TP, U3 STM32L072VZT6, U4 RNBD350, Y1 ABM8-272-T3

Commit message: updates to HIP and Controller design
Parts:
- removed C15: 4u7, Capacitor_SMD:C_0402_1005Metric_Pad0.74x0.62mm_HandSolder, symbol Device:C
- removed C18, C24: 100n, Capacitor_SMD:C_0402_1005Metric_Pad0.74x0.62mm_HandSolder, symbol Device:C
- removed D1: BLE, LED_SMD:LED_0805_2012Metric_Pad1.15x1.40mm_HandSolder, symbol Device:LED_Small_Filled
- removed J2: Conn_ARM_JTAG_SWD_10, Connector_PinHeader_1.27mm:PinHeader_2x05_P1.27mm_Vertical_SMD, symbol Connector:Conn_ARM_JTAG_SWD_10
- removed J4: BLE_DBG, Connector:Tag-Connect_TC2030-IDC-NL_2x03_P1.27mm_Vertical, symbol Connector:Conn_ARM_SWD_TagConnect_TC2030-NL
- removed R15, R17: 0R, Resistor_SMD:R_0402_1005Metric_Pad0.72x0.64mm_HandSolder, symbol Device:R
- removed R16: 330R, Resistor_SMD:R_0402_1005Metric_Pad0.72x0.64mm_HandSolder, symbol Device:R
- removed R23: 24.9k, Resistor_SMD:R_0402_1005Metric_Pad0.72x0.64mm_HandSolder, symbol Device:R
- removed SW3: BT_SCAN, Button_Switch_SMD:SW_SPST_EVQP7C, symbol Switch:SW_Push
- removed U4: RNBD350, pico_bldc:RNBD350, symbol RNBD350:RNBD350
- added J3: BLE_DBG, Connector:Tag-Connect_TC2030-IDC-NL_2x03_P1.27mm_Vertical, symbol Connector:Conn_ARM_SWD_TagConnect_TC2030-NL
- added J5: GND_Testpoint, Connector_PinSocket_2.54mm:PinSocket_1x02_P2.54mm_Vertical, symbol Connector_Generic:Conn_01x02
- added R13: 0R, Resistor_SMD:R_0402_1005Metric_Pad0.72x0.64mm_HandSolder, symbol Device:R
- added TP22, TP31, TP32, TP33, TP34, TP35, TP36: TestPoint, TestPoint:TestPoint_Pad_D1.0mm, symbol Connector:TestPoint
- added U3: BM71BLES1FC2-0B02AA, picostroke:BM71BLES1FC2_MCH, symbol BM71BLES1FC2:BM71BLES1FC2-0B02AA
- J4: renamed from J5; footprint picostroke:5037630491 -> Connector_PinHeader_2.00mm:PinHeader_1x04_P2.00mm_Vertical_SMD_Pin1Left
- renumbered C22 to C10, C14 to C12, C17 to C13, C23 to C14, C6 to C16, C7 to C17, C5 to C19, C8 to C20, C20 to C21, C12 to C22, C25 to C23, C4 to C25, C9 to C4, C10 to C5, C13 to C6, C16 to C7, C19 to C8, C21 to C9, J7 to J2, R12 to R10, R13 to R12, R20 to R14, R19 to R15, R24 to R19, R22 to R20, R9 to R22, R10 to R24, R14 to R5, R5 to R6, R6 to R9, U2 to U11, U3 to U2
Connections:
- net +3.3V: now also J3.1 (VCC), U3.14 (VBAT)
- net BLE_CTS: now also U3.11 (P0_0)
- net BLE_RTS: now also U3.9 (P3_6)
- net BLE_RX: now also TP32.1, U3.7 (HCI_RXD)
- net BLE_STAT1: now also U3.3 (P1_2)
- net BLE_STAT2: now also U3.4 (P1_3)
- net BLE_TX: now also TP31.1, U3.8 (HCI_TXD)
- net BLE_WAKEUP: now also U3.6 (P1_6)
- net GND: now also J3.5 (GND), J5.1 (Pin_1), J5.2 (Pin_2), R13.1, U3.13 (GND), U3.2 (GND); no longer J2.12
- net I2C0_SCL: now also TP36.1
- net I2C0_SDA: now also TP35.1
- net SWCLK: now also TP4.1
- net SWDIO: now also TP5.1
- net TX_ALRT: now also TP34.1, U3.15 (P2_7)
- net T_SWCLK: now also J3.4 (SWCLK); no longer TP4.1
- net T_SWDIO: now also J3.2 (SWDIO); no longer TP5.1
- net UART_MODE_SW: now also R13.2, U3.16 (P2_0)
- net ~{MRST}: now also TP33.1, U3.10 (RST_N)
- net ~{RESET}: now also J3.3 (~{RESET}), TP22.1
- net PS_VER: now reaches U2.35 (PB0)
- net +3.3VA renamed VDDA
- net AMB_I2C_INT renamed BATT_STAT
- net BLE_SW renamed BATT_~{CE}
- net BT_SIGNAL_GOOD renamed BATT_PG
- net LMAT_INT renamed KB_VER
- net LMAT_RST renamed HAPTIC_BRD_VER
- net HAPTIC_BRD_VER: now also J2.12
- no-connect marks 42 -> 34
Other:
- note added: "Bluetooth Low Energy Module BM71"
- note added: "Connectors"
- note removed: "Bluetooth Low Energy Module"
- note removed: "RNBD350 User Guide"
- company: (none) -> Yolk Workshop
- moved on the sheet: C16, C17, C19, C20, C21, C22, C23, R10, R11, R12, R14, R15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
