File: Yolk Workshop - Vitellus/PSU.kicad_sch (KiCad schematic)
At the start: 79 parts, among them Q2 BC859, Q3 PXP6R1-30QLJ, Q4 BC859, Q5 PXP6R1-30QLJ, Q6 BSN20BKR, SW4 POWER SW, U10 TPS6282533DMQR, U5 BQ25176JDSGR, U6 TXB0104PW, U7 MAX17055ETB+, U8 NCP380HMU15AATBG, U9 TPS630701RNMR

Commit message: updates to HIP and Controller design
Parts:
- removed C26, C31, C33: 1u, Capacitor_SMD:C_0402_1005Metric_Pad0.74x0.62mm_HandSolder, symbol Device:C
- removed C27, C28: 100n, Capacitor_SMD:C_0402_1005Metric_Pad0.74x0.62mm_HandSolder, symbol Device:C
- removed C29: 100n, Capacitor_SMD:C_0402_1005Metric_Pad0.74x0.62mm_HandSolder, symbol Device:C_Small
- removed D2: ON, LED_SMD:LED_0805_2012Metric, symbol Device:LED_Small
- removed D3: CHRG, LED_SMD:LED_0805_2012Metric, symbol Device:LED_Small
- removed D4: BAT_GOOD, LED_SMD:LED_0805_2012Metric, symbol Device:LED_Small
- removed D5: SYS_{PWR}, LED_SMD:LED_0603_1608Metric_Pad1.05x0.95mm_HandSolder, symbol Device:LED_Small
- removed Q2, Q4: BC859, Package_TO_SOT_SMD:SOT-23, symbol Transistor_BJT:BC859
- removed Q3, Q5: PXP6R1-30QLJ, pico_bldc:PXP01530QLJ, symbol PXP6R1-30QLJ:PXP6R1-30QLJ
- removed Q6: BSN20BKR, Package_TO_SOT_SMD:TSOT-23, symbol Simulation_SPICE:NMOS
- removed R25, R27: 3k6, Resistor_SMD:R_0402_1005Metric_Pad0.72x0.64mm_HandSolder, symbol Device:R_Small
- removed R37, R41: 10k, Resistor_SMD:R_0402_1005Metric_Pad0.72x0.64mm_HandSolder, symbol Device:R_Small
- removed R42: RT0402FRE0727K4L, Resistor_SMD:R_0402_1005Metric, symbol Device:R_Small
- removed R53: 1k, Resistor_SMD:R_0603_1608Metric, symbol Device:R_Small
- removed R8: 100k, Resistor_SMD:R_0402_1005Metric_Pad0.72x0.64mm_HandSolder, symbol Device:R_Small
- removed SW4: POWER SW, Button_Switch_SMD:SW_SPDT_PCM12, symbol Switch:SW_SPDT
- removed U5: BQ25176JDSGR, picostroke:SON50P200X200X80-9N, symbol BQ25176JDSGR:BQ25176JDSGR
- removed U6: TXB0104PW, Package_SO:TSSOP-14_4.4x5mm_P0.65mm, symbol Logic_LevelTranslator:TXB0104PW
- removed U8: NCP380HMU15AATBG, picostroke:UDFN6_2X2_ONS-L, symbol NCP380HMU15AATBG:NCP380HMU15AATBG
- added C15, C37, C48, C49: 4u7, Capacitor_SMD:C_0402_1005Metric_Pad0.74x0.62mm_HandSolder, symbol Device:C_Small
- added C18, C3, C38, C51: 1u, Capacitor_SMD:C_0402_1005Metric_Pad0.74x0.62mm_HandSolder, symbol Device:C_Small
- added C32, C33, C35: 100n, Capacitor_SMD:C_0402_1005Metric_Pad0.74x0.62mm_HandSolder, symbol Device:C_Small
- added C34: 47u, Capacitor_SMD:C_0805_2012Metric_Pad1.18x1.45mm_HandSolder, symbol Device:C_Small
- added C46, C47: 10u, Capacitor_SMD:C_0402_1005Metric_Pad0.74x0.62mm_HandSolder, symbol Device:C_Small
- added Q1: DMP3013SFV, Package_SON:Diodes_PowerDI3333-8, symbol Transistor_FET:DMP3013SFV
- added Q2: PMV13XN, Package_TO_SOT_SMD:SOT-23, symbol Transistor_FET:VN10LF
- added R16, R46: 100k, Resistor_SMD:R_0402_1005Metric_Pad0.72x0.64mm_HandSolder, symbol Device:R_Small
- added R17, R39: 27k4, Resistor_SMD:R_0402_1005Metric_Pad0.72x0.64mm_HandSolder, symbol Device:R_Small
- added R3, R4: 10k, Resistor_SMD:R_0402_1005Metric_Pad0.72x0.64mm_HandSolder, symbol Device:R_Small
- added R47, R48, R49: 2k2, Resistor_SMD:R_0402_1005Metric_Pad0.72x0.64mm_HandSolder, symbol Device:R_Small
- added TP10, TP16, TP17, TP18, TP21, TP23, TP25, TP26, TP27, TP28, TP29, TP8, TP9: TestPoint, TestPoint:TestPoint_Pad_D1.0mm, symbol Connector:TestPoint
- added U12: TS3333AQPR, picostroke:TS3333AQPR, symbol TS3333AQPR:TS3333AQPR
- added U13: MCP1252-33X50I_MS, picostroke:SOP65P490X110-8N, symbol MCP1252-33X50I_MS:MCP1252-33X50I_MS
- added U4: NCP380HMU15AATBG, picostroke:UDFN6_2X2_ONS-L, symbol NCP380HMU15AATBG:NCP380HMU15AATBG
- added U5: TPS2116DRL, Package_TO_SOT_SMD:SOT-583-8, symbol Power_Management:TPS2116DRL
- added U7: LPV7215MG_NOPB, picostroke:SOT65P210X110-5N, symbol LPV7215MG_NOPB:LPV7215MG_NOPB
- added U8: BQ25176JDSGR, picostroke:SON50P200X200X80-9N, symbol BQ25176JDSGR:BQ25176JDSGR
- C26: renamed from C36; footprint Capacitor_SMD:C_0402_1005Metric_Pad0.74x0.62mm_HandSolder -> Capacitor_SMD:C_0603_1608Metric_Pad1.08x0.95mm_HandSolder
- R26: value 3k6 -> 100k
- R28: value RC0402DR-0730KL -> 100k; footprint Resistor_SMD:R_0402_1005Metric -> Resistor_SMD:R_0402_1005Metric_Pad0.72x0.64mm_HandSolder; Val 30k -> (none)
- R29: value RT0402FRE0727K4L -> 100k; footprint Resistor_SMD:R_0402_1005Metric -> Resistor_SMD:R_0402_1005Metric_Pad0.72x0.64mm_HandSolder; Val 27k4 -> (none)
- R31, R34: value 2k2 -> 100k
- R32: value 2k2 -> 47k
- R33: value 10k -> 100k
- R35: value 10k -> 1.8M
- R36: value 2k2 -> 95k; now not fitted
- R38: value 10k -> 1K2
- R40: value 1k -> 25k; now not fitted
- R43, R44: value 1k -> 100k
- R45: value 1k -> 47k
- TH1: footprint Connector_PinHeader_2.54mm:PinHeader_1x02_P2.54mm_Vertical -> Connector_PinHeader_1.27mm:PinHeader_1x02_P1.27mm_Vertical
- renumbered C34 to C24, C38 to C27, C41 to C28, C42 to C29, C44 to C30, C46 to C31, C39 to C36, C40 to C39, C43 to C40, C45 to C41, C47 to C42, C35 to C43, C37 to C44, C30 to C45, C32 to C50, JP2 to JP1, L2 to L1, L1 to L2, R48 to R23, R49 to R25, R51 to R27, R46 to R37, R47 to R41, R52 to R42, R39 to R50, R50 to R8, TP10 to TP19, TP8 to TP20, TP9 to TP24, U7 to U10, U9 to U6, U10 to U9
Connections:
- net BAT_STAT_G is gone; now on net +3.3VA: R44.2
- net BAT_TS is gone; now on net BATT_TS: TH1.1
- net PNP_DIFF_BASE is gone; now on net ~{BATT_EN}: R35.1
- net VBUS_GATE is gone; now on net GND: R38.2
- net +1V8: no longer R31.2, R32.1, R34.1, R36.1
- net +3.3V: now also R47.2, R48.2, R49.2; no longer R26.2
- net BB_PG: now also TP9.1
- net BMS_ALRT: now also U10.8 (ALRT), R49.1
- net BMS_SCL: now also U10.3 (SCL), R48.1; no longer R26.1
- net BMS_SDA: now also U10.4 (SDA), R47.1
- net GND: now also C45.1, R26.1, R32.1, R34.2, R40.1, R45.1, C15.2, C18.2, C3.1, C32.2, C33.1, C34.2, C35.2, C37.2, C38.2, C46.1, C47.1, C48.2, C49.2, Q2.2 (S), R16.2, R17.1, R39.2, U12.4 (GND), U13.4 (GND), U13.8 (SELECT), U4.5 (GND), U4.7 (EPAD), U5.1 (GND), U7.2 (V-), U8.4 (GND), U8.9 (EPAD); no longer C45.2, R28.2, R29.2, R30.2, R35.2, R38.1
- net VBAT: now also C45.2, R31.1, C37.1, C46.2, Q1.1 (S), Q1.2 (S), Q1.3 (S), TP18.1, U13.3 (VIN), U13.7 (~{SHDN}), U8.8 (OUT); no longer C45.1, R43.1, R45.1
- net VBUS: now also C15.1, C18.1, C38.1, R4.1, U5.3 (VIN1), U5.5 (MODE), U8.1 (IN)
- net VDD: now also R29.2, R36.1, TP7.1, C3.2, C34.1, R3.1, U4.6 (IN), U5.2 (VOUT), U5.7 (VOUT); no longer TP6.1
- net VSYS: now also TP8.1, U4.1 (OUT); no longer R40.1, TP7.1
- net ~{BUCK_PG}: now also TP23.1
- net +BATT: now reaches BT1.1 (+), F2.1
- net -BATT: now reaches BT1.2 (-), C50.2, R50.2, TH1.2, U10.1 (N.C.), U10.11 (EP), U10.2 (AIN), U10.6 (CSP)
- net BATT_~{CE}: now reaches R45.2
- net BATT_~{CE}: now also Q2.1 (G)
- net BATT_PG: now reaches R43.2
- net BATT_PG: now also TP26.1, U8.6 (PG)
- net BATT_TS: now reaches R40.2
- net BATT_TS: now also R36.2, Q2.3 (D), TP21.1, U8.3 (TS)
- net BAT_ISET renamed +3.3VA
- net +3.3VA: now also R30.1, R43.1, C49.1, TP28.1, U12.8 (OUT)
- net BAT_STAT renamed BATT_STAT
- net BATT_STAT: now also TP25.1, U8.5 (STAT)
- net BAT_VSET renamed PL_FLAG
- net PL_FLAG: now also TP10.1, U4.3 (~{FLAG})
- net I2C_ALRT_1V8 renamed ~{BATT_EN}
- net ~{BATT_EN}: now also C35.1, Q1.4 (G), TP16.1, U7.1 (VOUT); no longer U10.8 (ALRT)
- removed net I2C_SCL_1V8: R34.2, U10.3 (SCL)
- removed net I2C_SDA_1V8: R36.2, U10.4 (SDA)
- removed net OE_1V8: R30.1, R31.1
- net VBAT_GATE renamed B_EN_VREF
- net B_EN_VREF: now also R30.2, R35.2, U7.3 (VIN+)
- new net: Q1.5 (D), U5.6 (VIN2)
- new net: R46.2, TP29.1, U13.1 (PGOOD)
- new net +5VA: C33.2, C47.2, C48.1, R46.1, TP27.1, U12.5 (IN), U13.2 (VOUT), U7.5 (V+)
- new net ISET: R38.1, U8.2 (ISET)
- new net PL_ILIM: R17.2, U4.2 (ILIM)
- new net PR: R16.1, R4.2, U5.4 (PR1)
- new net PWR_SW_A: R3.2
- new net PWR_SW_B: C32.1, R26.2, TP6.1, U4.4 (EN)
- new net VBATT_REF: R31.2, R34.1, U7.4 (VIN-)
- new net VBUS_DET: R28.2, TP17.1, U5.8 (ST)
- new net VSET: R39.1, U8.7 (VSET)
- new net c+: C51.2, U13.6 (C+)
- new net c-: C51.1, U13.5 (C-)
- no-connect marks 4 -> 1
Other:
- note added: "Auto Power Multiplexer"
- note added: "Auxillary Power & Voltage Reference"
- note added: "Battery Discharge Protection"
- note added: "Coulomb Counter"
- note removed: "AUTO-POWER SWITCHER"
- note removed: "Auto-Power Switcher Disconnects V_{BAT} when V_{BUS} is detected"
- note removed: "BATTERY CHARGER"
- note removed: "BATTERY MONITOR"
- note removed: "Battery Specifications"
- note removed: "Charge Indicator"
- note removed: "Charger Indicators LED Red := Charge in progress LED Green := charge complete/ disabled LED Red [blink] (1 sec) := Fault Condition"
- note removed: "I_{CHG} := 30k ~100mA I_{TERM} := 100*0.1 - 10mA I_{PRECHG} := 100*0.2 - 20mA"
- note removed: "I_{SET} := 30k"
- note removed: "V_{SET} := 27k4 V_{CHG} := 4V2"
- company: Yolk workshop -> Yolk Workshop
- moved on the sheet: BT1, C24, C26, C27, C28, C29, C30, C31, C45, C50, F2, R50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
