File: Yolk Workshop - Vitellus/USB.kicad_sch (KiCad schematic)
At the start: 15 parts, among them J1 USB4105-GF-A, Q1 PMV13XN, U1 USBLC6-2SC6

Commit message: updates to HIP and Controller design
Parts:
- removed C3: 100n, Capacitor_SMD:C_0402_1005Metric_Pad0.74x0.62mm_HandSolder, symbol Device:C_Small
- removed Q1: PMV13XN, Package_TO_SOT_SMD:SOT-23, symbol Transistor_FET:VN10LF
- removed R3, R4: 47k, Resistor_SMD:R_0603_1608Metric_Pad0.98x0.95mm_HandSolder, symbol Device:R_Small
Other:
- company: (none) -> Yolk Workshop
- moved on the sheet: C1, C2, F1, J1, R1, R2, R7, TP1, TP2, TP3
